File: TSAL copy.kicad_pcb (KiCad board)
At the start: 2 copper layers, 87 x 52 mm, 55 parts, among them J1 Conn_01x02_Socket, J10 Conn_01x02_Socket, J11 Conn_01x02_Socket, J12 Conn_01x02_Socket, J13 Conn_01x02_Socket, J14 Conn_01x02_Socket, J15 Conn_01x02_Socket, J2 Conn_01x02_Socket, J3 Conn_01x02_Socket, J4 Conn_01x02_Socket, J5 Conn_01x02_Socket, J6 Conn_01x02_Socket, J7 Conn_01x02_Socket, J8 Conn_01x02_Socket, J9 Conn_01x02_Socket, Q1 AO3401A, Q3 AO3401A, Q4 AO3400A, U1 AMC0380R4, U12 TLV2372, U13 74AHC1G04, U14 74AHCT1G02, U15 74AHC04, U16 74AHC1G04, U2 LT6995-1, U3 TMA-0505S, U4 74HC00, U5 74AHC2G00, U7 74AHC1G08, U8 74AHCT1G02, U9 74HC86

Commit message: AddedPullDown
Parts:
- moved U3 4.52 mm to (137.6, 91.1)
Routing:
- net Net-(J14-Pin_1): track 37.3 -> 34.2 mm
- net Net-(J14-Pin_2): track 41.1 -> 39.8 mm
- net Net-(U1-VDD1): track 40.3 -> 41.6 mm
- net Net-(J15-Pin_1): track 61.5 -> 62.8 mm
Other:
- board text added: "HV Input"
