File: TSAL copy.kicad_sch (KiCad schematic)
At the start: 20 parts, among them Q1 PMOS, Q2 PMOS, Q3 NMOS, U1 AMC0380R4, U2 TLC555xD, U3 TMA-0505S, U4 LM311, U5 74LVC1G11

Commit message: AddedPullDown
Parts:
- removed Q1, Q2: PMOS, symbol Simulation_SPICE:PMOS
- removed Q3: NMOS, symbol Simulation_SPICE:NMOS
- removed U2: TLC555xD, Package_SO:SOIC-8_3.9x4.9mm_P1.27mm, symbol Timer:TLC555xD
- removed U4: LM311, symbol Comparator:LM311
- removed U5: 74LVC1G11, symbol 74xGxx:74LVC1G11
- added C5: 100n, 100n:CAPC3216X95N, symbol Device:C
- added C6: 1u, 1u:1206_AVX, symbol Device:C
- added D1, D2, D3, D4, D5, D6, D7, D8: LED, LED:LEDC1608X70N, symbol Device:LED
- added J1, J10, J11, J12, J13, J14, J15, J16, J2, J3, J4, J5, J6, J7, J8, J9: Conn_01x02_Socket, JST-B02B-PASK:B02BPASK1LFSN, symbol Connector:Conn_01x02_Socket
- added Q1, Q3: AO3401A, Package_TO_SOT_SMD:SOT-23, symbol Transistor_FET:AO3401A
- added Q4: AO3400A, Package_TO_SOT_SMD:SOT-23, symbol Transistor_FET:AO3400A
- added R10, R11, R13, R14, R9: 1k, 1k:RESC3116X65N, symbol Device:R
- added R12: R, symbol Device:R
- added U10, U12: TLV2372, TLV0732:SOP65P490X110-8N, symbol Amplifier_Operational:TLV2372
- added U11, U13, U16: 74AHC1G04, SN74AHC1G04QDBVRQ1:DBV5, symbol 74xGxx:74AHC1G04
- added U14, U8: 74AHCT1G02, SN74AHCT1G02:DBV5, symbol 74xGxx:74AHCT1G02
- added U15: 74AHC04, SN74AHC04:D14, symbol 74xx:74AHC04
- added U17: TPS259474LRPWR, RPW0010A-MFG, symbol TPS25947LRPWR:TPS259474LRPWR
- added U2: LT6995-1, LTC6995-1:SOT95P280X100-6N, symbol LTC6995-1:LTC6995-1
- added U4: 74HC00, 74HC00:SOIC127P600X175-14N, symbol 74xx:74HC00
- added U5: 74AHC2G00, 74AHC2G00:SOP50P310X100-8N, symbol 74xGxx:74AHC2G00
- added U6: AMC0380R4, AMC0380R4:AMC0380R04DFXR, symbol AMC0380R4:AMC0380R4
- added U7: 74AHC1G08, SN74AHC1G08QDBVRQ1:DBV5, symbol 74xGxx:74AHC1G08
- added U9: 74HC86, SN74HC86:PW14, symbol 74xx:74HC86
- C1: value 10n -> 1u; footprint (none) -> 1u:1206_AVX
- C2: value 10u -> 100n; footprint (none) -> 100n:CAPC3216X95N
- C3, C4: value C -> 100p; footprint (none) -> 100p:C1206
- R1: value 1K -> 976k; footprint (none) -> 976k:RC1206N_YAG
- R2: value 17.5K -> 187k; footprint (none) -> 976k:RC1206N_YAG
- R3: value 20K -> 191k; footprint (none) -> 976k:RC1206N_YAG
- R4: value 8.3M -> 1k; footprint (none) -> 1k:RESC3116X65N
- R5: value 20.8K -> 1k; footprint (none) -> 1k:RESC3116X65N
- R6, R7: value 500K -> 1k; footprint (none) -> 1k:RESC3116X65N
- R8: value R -> 1k; footprint (none) -> 1k:RESC3116X65N
- U1: footprint (none) -> AMC0380R4:AMC0380R04DFXR
Connections:
- net at C4.1: now also C1.1, C2.1, C3.1, U1.2 (SNSC), U1.6 (GND1), U3.4 (-Vout), C5.1, C6.1, J15.1 (Pin_1), J16.1 (Pin_1), U6.2 (SNSC), U6.6 (GND1); no longer U1.
- net at R8.2: now also D3.2 (A)
- net at C1.2: now also C2.2, U1.5 (VDD1), U3.6 (+Vout), C6.2, U6.5 (VDD1)
- net at R4.1: now also U2.4 (OUT)
- net at R5.1: now also Q1.2 (S); no longer R4.2
- net at R5.2: now also J13.1 (Pin_1), Q4.3 (D)
- net GND: now reaches R2.2
- net GND: now also R3.2, U1.9 (GND2), D1.1 (K), D2.1 (K), D3.1 (K), D4.1 (K), D5.1 (K), D6.1 (K), D7.1 (K), D8.1 (K), J1.2 (Pin_2), J10.2 (Pin_2), J11.2 (Pin_2), J12.2 (Pin_2), J13.2 (Pin_2), J2.2 (Pin_2), J3.2 (Pin_2), J4.2 (Pin_2), J5.2 (Pin_2), J6.2 (Pin_2), J7.2 (Pin_2), J8.2 (Pin_2), J9.2 (Pin_2), Q4.2 (S), R12.2, U10.4 (V-), U11.3 (GND), U12.4 (V-), U13.3 (GND), U14.3 (GND), U15.7 (GND), U16.3 (GND), U2.5 (GND), U2.6 (RST), U4.7 (GND), U5.4 (GND), U6.9 (GND2), U7.3 (GND), U8.2, U8.3 (GND), U9.7 (GND); no longer C2.1
- net +5V: now reaches R1.1
- net +5V: now also U1.11 (REFIN), U1.14 (VDD2), Q3.3 (D), U10.8 (V+), U12.8 (V+), U6.11 (REFIN), U6.14 (VDD2); no longer R3.2
- net at R6.1: now also U16.4, U4.4
- net at R1.2, R2.1: now also U2.2 (DIV)
- removed net GLV+: R3.1, R7.2, R8.1, U1., U3.1 (+Vin)
- removed net GLV-: C1.1, C2.2, R6.2, R7.1, U1., U3.2 (-Vin)
- new net: D6.2 (A), R14.1
- new net: Q4.1 (G), R12.1, U14.2, U8.4
- new net: R14.2, U15.6, U5.6
- new net: D2.2 (A), R7.1
- new net: R7.2, U10.1, U4.10, U9.13
- new net: U15.5, U9.8
- new net: J8.1 (Pin_1), U9.5
- new net: D1.2 (A), R6.2
- new net: C3.2, U1.4 (SNSP)
- new net: J14.2 (Pin_2), U3.1 (+Vin)
- new net: J14.1 (Pin_1), U3.2 (-Vin)
- new net: Q1.1 (G), U4.6
- new net: D7.2 (A), R11.1
- new net: R11.2, U15.8, U7.2
- new net: U12.1, U4.1
- new net: U1.10 (OUT), U12.3 (+)
- new net: J6.1 (Pin_1), U9.4
- new net: U15.3, U9.6
- new net: U11.2, U7.4
- new net: U11.4, U14.1
- new net: U13.2, U4.8
- new net: U13.4, U4.5
- new net: J10.1 (Pin_1), U9.10
- new net: J7.1 (Pin_1), U9.9
- new net: J4.1 (Pin_1), R8.1, U4.9
- new net: U10.3 (+), U6.10 (OUT)
- new net: U15.11, U5.3
- new net: U15.12, U5.5
- new net: Q3.1 (G), R13.2, U4.3
- new net: Q3.2 (S), U2.1 (V)
- new net: R3.1, U2.3 (SET)
- new net: U15.9, U9.11
- new net: J11.1 (Pin_1), U9.12
- new net: D8.2 (A), R13.1
- new net: J12.1 (Pin_1), R4.2
- new net: U16.2, U4.11
- new net: J2.1 (Pin_1), U4.13
- new net: J5.1 (Pin_1), U9.1
- new net: U15.10, U7.1
- new net: R9.1, U15.2, U5.1
- new net: D4.2 (A), R9.2
- new net: R10.2, U15.4, U5.2
- new net: U15.13, U5.7
- new net: J9.1 (Pin_1), U9.2
- new net: J15.2 (Pin_2), U1.1 (HVIN)
- new net: U14.4, U8.1
- new net: J3.1 (Pin_1), U4.12
- new net: J16.2 (Pin_2), U6.1 (HVIN)
- new net: C4.2, U6.4 (SNSP)
- new net: U15.1, U9.3
- new net: D5.2 (A), R10.1
- new net: J1.1 (Pin_1), U4.2
- new net 0.75V: U10.2 (-), U12.2 (-)
- new net VCC: Q1.3 (D), U11.5 (VCC), U13.5 (VCC), U14.5 (VCC), U15.14 (VCC), U16.5 (VCC), U4.14 (VCC), U5.8 (VCC), U7.5 (VCC), U8.5 (VCC), U9.14 (VCC)
- no-connect marks 0 -> 7
Other:
- note added: "AIR 1"
- note added: "AIR 1 Open"
- note added: "AIR 2"
- note added: "AIR 2 Open"
- note added: "Add another Multi-input NOR gate for all the relays"
- note added: "From HV Sensing Circuit (Above 60V results in HIGH)"
- note added: "From VCU (In case of any SCS failure, results in LOW)"
- note added: "GLV+"
- note added: "GLV-"
- note added: "Green Light Activation Circuit"
- note added: "High Voltage Sensing Signal (If below 60V, LOW)"
- note added: "Implement using resistor divider"
- note added: "Intentional AIR 1 (From VCU)"
- note added: "Intentional AIR 2 (From VCU)"
- note added: "Intentional Precharge (From VCU)"
- note added: "Make active high"
- note added: "Precharge"
- note added: "Precharge Relay Open"
- note added: "R"
- note added: "Red Light Activation"
- note added: "S"
- note added: "Safe State Activation Circuit"
- note added: "Signal from Comparator"
- note added: "Voltage High or Low Signal From VCU"
- note removed: "HV"
- note removed: "LV"
- note removed: "Signals from other modules"
- moved on the sheet: U3
