File: TSAL.kicad_sch (KiCad schematic)
At the start: 55 parts, among them J1 Conn_01x02_Socket, J10 Conn_01x02_Socket, J11 Conn_01x02_Socket, J12 Conn_01x02_Socket, J13 Conn_01x02_Socket, J14 Conn_01x02_Socket, J15 Conn_01x02_Socket, J2 Conn_01x02_Socket, J3 Conn_01x02_Socket, J4 Conn_01x02_Socket, J5 Conn_01x02_Socket, J6 Conn_01x02_Socket, J7 Conn_01x02_Socket, J8 Conn_01x02_Socket, J9 Conn_01x02_Socket, Q1 AO3401A, Q3 AO3401A, Q4 AO3400A, U1 AMC0380R4, U12 TLV2372, U13 74AHC1G04, U14 74AHCT1G02, U15 74AHC04, U16 74AHC1G04, U2 LT6995-1, U3 TMA-0505S, U4 74HC00, U5 74AHC2G00, U7 74AHC1G08, U8 74AHCT1G02, U9 74HC86

Commit message: AddedPullDown
Parts:
- added C4: 100p, 100p:C1206, symbol Device:C
- added C5: 100n, 100n:CAPC3216X95N, symbol Device:C
- added C6: 1u, 1u:1206_AVX, symbol Device:C
- added J16: Conn_01x02_Socket, JST-B02B-PASK:B02BPASK1LFSN, symbol Connector:Conn_01x02_Socket
- added U10: TLV2372, TLV0732:SOP65P490X110-8N, symbol Amplifier_Operational:TLV2372
- added U6: AMC0380R4, AMC0380R4:AMC0380R04DFXR, symbol AMC0380R4:AMC0380R4
Connections:
- net +5V: now also U10.8 (V+), U6.11 (REFIN), U6.14 (VDD2)
- net 0.75V: now also U10.2 (-)
- net GND: now also U10.4 (V-), U6.9 (GND2)
- net at C1.1, C2.1, C3.1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: now also C4.1, C5.1, C6.1, J16.1 (Pin_1), U6.2 (SNSC), U6.6 (GND1)
- net at C1.2, C2.2, U1.5 (VDD1)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: now also C6.2, U6.5 (VDD1)
- net at R7.2, U4.10, U9.13: now also U10.1; no longer U12.1, U4.1
- new net: U12.1, U4.1
- new net: U10.3 (+), U6.10 (OUT)
- new net: J16.2 (Pin_2), U6.1 (HVIN)
- new net: C4.2, U6.4 (SNSP)
- no-connect marks 4 -> 7
Other:
- note added: "Add another Multi-input NOR gate for all the relays"
- note added: "Implement using resistor divider"
- note added: "Make active high"
- moved on the sheet: U15G, U9E
